File: hapticDriver/hapticDriver/hapticDriver.kicad_sch (KiCad schematic)
At the start: 15 parts, among them J1 AudioJack2, J3 AudioJack2, U1 TL074, U2 LD1117V33

Commit message: new
Parts:
- removed C1: 10µF, symbol Device:C
- removed D1: 1N4148, Diode_THT:D_DO-35_SOD27_P7.62mm_Horizontal, symbol Diode:1N4148
- removed D3: 1N5817, Diode_THT:D_DO-41_SOD81_P10.16mm_Horizontal, symbol Diode:1N5817
- removed J3: AudioJack2, symbol Connector_Audio:AudioJack2
- removed MES1: VOLTMETER_DIFF, symbol Simulation_SPICE:VOLTMETER_DIFF
- removed R1: 10MΩ, symbol Device:R_US
- removed U2: LD1117V33, Package_TO_SOT_THT:TO-220-3_Vertical, symbol Regulator_Linear:LD1117V33
- removed V1: VSIN, symbol Simulation_SPICE:VSIN
- removed V2: 12, symbol Simulation_SPICE:VDC
- added D1: 1N5817, Diode_THT:D_DO-41_SOD81_P10.16mm_Horizontal, symbol Diode:1N5817
- added Gain: 1K, symbol Device:R_Potentiometer_US
- added J2: AudioJack2, symbol Connector_Audio:AudioJack3
- added R4, R5: 1K, symbol Device:R_US
- added R6: 10K, symbol Device:R_US
- R1: renamed from R4; value 10kΩ -> 1M
- R2: value 1kΩ -> 330
- R3: value 1kΩ -> 470
Connections:
- net GND: now also R1.2, R2.2, U1.12 (+), Gain.3, J2.S, R6.2; no longer R3.2
- net at J1.T: now also U1.10 (+), R6.1
- net at U1.1, U1.2 (-): now also D1.2 (A)
- net at R1.1: now also U1.5 (+), Gain.2
- net at R3.1, U1.3 (+): now also U1.7, R4.2; no longer R2.2
- net at R2.1: now also R3.2, U1.6 (-)
- net at U1.13 (-): now also R4.1, R5.2
- net at U1.14: now also D2.2 (A), R5.1
- net at U1.8: now also U1.9 (-), Gain.1
- net +3.3V: no longer names the net of D2.1 (K)
- net +3.3V: now also J2.R
- net 0 renamed -12V
- new net: D1.1 (K), J2.T
Other:
- note added: "(Eurorack IDC)"
- note added: "(amplifier)"
- note added: "(buffer)"
- note added: "(inverter)"
- note added: "from CV source (front plate - TS)"
- note added: "front plate"
- note added: "gain control (front plate - knob)"
- note added: "negative buzzer"
- note added: "positive buzzer"
- note added: "to ERM motor (front plate - TRS)"
- note removed: "3.3V"
- note removed: "from CV source"
- note removed: "to ERM motor"
- title: (none) -> SynthAccess Haptic Driver
- moved on the sheet: R1, U1A, U1B, U1C, U1D, U1E
